Commit message: [Somewhere]

File: mobile_manipulator_body/urdf/mobile_manipulator.urdf (robot description, URDF)
Before this commit: robot mobile_manipulator, 10 links, 9 joints
Links:
- added link camera_link, mass 1e-5; collision box size=0.05 0.05 0.05; visual box size=0.05 0.05 0.05
- added link imu_link, mass 0.001; collision box size=.001 .001 .001; visual box size=0.001 0.001 0.001
- added link laser_link, mass 1e-5; collision box size=0.1 0.1 0.1; visual box size=0.05 0.05 0.05
- link base_link: mass 47.873 -> 48.0
Joints:
- added joint camera_joint: type fixed, parent base_link, child camera_link, origin xyz=0.25 0 0.185 rpy=0 0 0, axis 0 1 0
- added joint imu_joint: type fixed, parent base_link, child imu_link, origin xyz=-0.350 0 0.115, axis 1 0 0
- added joint laser_joint: type fixed, parent base_link, child laser_link, origin xyz=0.350 0 0.115 rpy=0 0 0, axis 0 1 0

File: mobile_manipulator_body/urdf/robot_base.urdf (robot description, URDF)
Before this commit: robot robot_base, 7 links, 6 joints
Links:
- removed link camera_link
- removed link camera_link_optical
- added link laser_link, mass 1e-5; collision box size=0.1 0.1 0.1; visual box size=0.05 0.05 0.05
Joints:
- removed joint camera_joint
- removed joint camera_optical_joint
- added joint laser_joint: type fixed, parent base_link, child laser_link, origin xyz=0.350 0 0.115 rpy=0 0 0, axis 0 1 0
