Commit message: [Top View Camera Added]

File: mobile_manipulator/urdf/mobile_manipulator.urdf (robot description, URDF)
Before this commit: robot mobile_manipulator, 13 links, 12 joints
Links:
- removed link camera_link
- added link front_camera_link, mass 1e-5; collision box size=0.05 0.05 0.05; visual box size=0.05 0.05 0.05
Joints:
- removed joint camera_joint
- added joint front_camera_joint: type fixed, parent base_link, child front_camera_link, origin xyz=0.25 0 0.185 rpy=0 0 0, axis 0 1 0
